File: Power management board/cosi_pwr.kicad_pcb (KiCad board)
At the start: 2 copper layers, 118.4 x 104.3 mm, 54 parts, among them K1 PT371512, K2 G5SB, U1 IRM_15_20, U10 N-CHANNEL-MOSFET-BSS138, U11 N-CHANNEL-MOSFET-BSS138, U2 DCDC_SIM1_DIP8, U3 N-CHANNEL-MOSFET-BSS138, U5 N-CHANNEL-MOSFET-BSS138, U6 N-CHANNEL-MOSFET-BSS138, U7 N-CHANNEL-MOSFET-BSS138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

Commit message: Adding info for electronics and casing design
Other:
- net class Default removed
- net class ac removed
- net class power removed
